File: 2Buttons_Input.kicad_pcb (KiCad board)
At the start: 2 copper layers, 46.2 x 30.2 mm, 19 parts, among them J1 JST_SH_SM06B-SRSS-TB_1x06-1MP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, SW1 SW_Push, SW2 SW_Push, U1 M24C02-FMN

Commit message: Change I2C pull-up resistors value to 4.7K
Parts:
- R5, R6: value 2.2K -> 4.7K
