File: 2Buttons_Input.kicad_sch (KiCad schematic)
At the start: 13 parts, among them J1 JST_SH_SM06B-SRSS-TB_1x06-1MP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, SW1 SW_Push, SW2 SW_Push, U1 M24C02-FMN

Commit message: Change I2C pull-up resistors value to 4.7K
Parts:
- R5, R6: value 2.2K -> 4.7K
Changed lines of the file:
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@@
 (kicad_sch
-	(version 20231120)
+	(version 20250114)
 	(generator "eeschema")
-	(generator_version "8.0")
+	(generator_version "9.0")
 	(paper "A5")
 	(title_block
@@
 		(company "A.B. Yazamut")
 	)
+	(rectangle
+		(start 13.335 14.605)
+		(end 89 74.93)
+		(stroke
+			(width 0)
+			(type dash)
+		)
+		(fill
+			(type none)
+		)
+	)
+	(rectangle
+		(start 90.8 62.23)
+		(end 168 100.33)
+		(stroke
+			(width 0)
+			(type dash)
+		)
+		(fill
+			(type none)
+		)
+	)
+	(rectangle
+		(start 13.335 76.835)
+		(end 89 100.33)
+		(stroke
+			(width 0)
+			(type dash)
+		)
+		(fill
+			(type none)
+		)
+	)
+	(rectangle
+		(start 90.8 14.605)
+		(end 168 60.96)
+		(stroke
+			(width 0)
+			(type dash)
+		)
+		(fill
+			(type none)
+		)
+	)
+	(text "EEPROM"
+		(exclude_from_sim no)
+		(at 92.075 17.78 0)
+		(effects
+			(font
+				(size 1.27 1.27)
+			)
+			(justify left bottom)
+		)
+	)
+	(text "Connectors"
+		(exclude_from_sim no)
+		(at 92.456 65.786 0)
+		(effects
+			(font
+				(size 1.27 1.27)
+			)
+			(justify left bottom)
+		)
+	)
+	(text "I2C Pull-UPs"
+		(exclude_from_sim no)
+		(at 14.224 80.01 0)
+		(effects
+			(font
+				(size 1.27 1.27)
+			)
+			(justify left bottom)
+		)
+	)
+	(text "Debounce"
+		(exclude_from_sim no)
+		(at 14.478 17.78 0)
+		(effects
+			(font
+				(size 1.27 1.27)
+			)
+			(justify left bottom)
+		)
+	)
 	(junction
 		(at 114.3 46.99)
@@
 			(width 0)
 			(type default)
-		)
-	)
-	(rectangle
-		(start 13.335 14.605)
-		(end 89 74.93)
-		(stroke
-			(width 0)
-			(type dash)
-		)
-		(fill
-			(type none)
-		)
-	)
-	(rectangle
-		(start 90.8 62.23)
-		(end 168 100.33)
-		(stroke
-			(width 0)
-			(type dash)
-		)
-		(fill
-			(type none)
-		)
-	)
-	(rectangle
-		(start 13.335 76.835)
-		(end 89 100.33)
-		(stroke
-			(width 0)
-			(type dash)
-		)
-		(fill
-			(type none)
-		)
-	)
-	(rectangle
-		(start 90.8 14.605)
-		(end 168 60.96)
-		(stroke
-			(width 0)
-			(type dash)
-		)
-		(fill
-			(type none)
-		)
-	)
-	(text "EEPROM"
-		(exclude_from_sim no)
-		(at 92.075 17.78 0)
-		(effects
-			(font
-				(size 1.27 1.27)
-			)
-			(justify left bottom)
-		)
-	)
-	(text "Connectors"
-		(exclude_from_sim no)
-		(at 92.456 65.786 0)
-		(effects
-			(font
-				(size 1.27 1.27)
-			)
-			(justify left bottom)
-		)
-	)
-	(text "I2C Pull-UPs"
-		(exclude_from_sim no)
-		(at 14.224 80.01 0)
-		(effects
-			(font
-				(size 1.27 1.27)
-			)
-			(justify left bottom)
-		)
-	)
-	(text "Debounce"
-		(exclude_from_sim no)
-		(at 14.478 17.78 0)
-		(effects
-			(font
-				(size 1.27 1.27)
-			)
-			(justify left bottom)
 		)
 	)
@@
 		)
 		(instances
-			(project "QWIIC_adapter"
+			(project "2Buttons_Input"
 				(path "/1a1c72da-99f5-4976-b608-38ee505f2b67"
 					(reference "#PWR06")
@@
 		)
 		(instances
-			(project "QWIIC_adapter"
+			(project "2Buttons_Input"
 				(path "/1a1c72da-99f5-4976-b608-38ee505f2b67"
 					(reference "#PWR03")
@@
 			)
 		)
-		(property "Value" "2.2K"
+		(property "Value" "4.7K"
 			(at 30.48 84.836 90)
 			(effects
@@
 		)
 		(instances
-			(project ""
+			(project "2Buttons_Input"
 				(path "/1a1c72da-99f5-4976-b608-38ee505f2b67"
 					(reference "R5")
@@
 		)
 		(instances
-			(project "QWIIC_adapter"
+			(project "2Buttons_Input"
 				(path "/1a1c72da-99f5-4976-b608-38ee505f2b67"
 					(reference "#PWR04")
@@
 		)
 		(instances
-			(project "QWIIC_adapter"
+			(project "2Buttons_Input"
 				(path "/1a1c72da-99f5-4976-b608-38ee505f2b67"
 					(reference "#FLG01")
@@
 		)
 		(instances
-			(project "QWIIC_adapter"
+			(project "2Buttons_Input"
 				(path "/1a1c72da-99f5-4976-b608-38ee505f2b67"
 					(reference "#PWR01")
@@
 		)
 		(instances
-			(project ""
+			(project "2Buttons_Input"
 				(path "/1a1c72da-99f5-4976-b608-38ee505f2b67"
 					(reference "R2")
@@
 		)
 		(instances
-			(project "QWIIC_adapter"
+			(project "2Buttons_Input"
 				(path "/1a1c72da-99f5-4976-b608-38ee505f2b67"
 					(reference "#FLG02")
@@
 		)
 		(instances
-			(project ""
+			(project "2Buttons_Input"
 				(path "/1a1c72da-99f5-4976-b608-38ee505f2b67"
 					(reference "C2")
@@
 		)
 		(instances
-			(project "QWIIC_adapter"
+			(project "2Buttons_Input"
 				(path "/1a1c72da-99f5-4976-b608-38ee505f2b67"
 					(reference "C1")
@@
 		)
 		(instances
-			(project "SAMD21_Dev_Board"
+			(project "2Buttons_Input"
 				(path "/1a1c72da-99f5-4976-b608-38ee505f2b67"
 					(reference "#PWR014")
@@
 			)
 		)
-		(property "Value" "2.2K"
+		(property "Value" "4.7K"
 			(at 30.48 94.488 90)
 			(effects
@@
 		)
 		(instances
-			(project ""
+			(project "2Buttons_Input"
 				(path "/1a1c72da-99f5-4976-b608-38ee505f2b67"
 					(reference "R6")
@@
 		)
 		(instances
-			(project "QWIIC_adapter"
+			(project "2Buttons_Input"
 				(path "/1a1c72da-99f5-4976-b608-38ee505f2b67"
 					(reference "#PWR05")
@@
 		)
 		(instances
-			(project "QWIIC_adapter"
+			(project "2Buttons_Input"
 				(path "/1a1c72da-99f5-4976-b608-38ee505f2b67"
 					(reference "U1")
@@
 		)
 		(instances
-			(project "SAMD21_Dev_Board"
+			(project "2Buttons_Input"
 				(path "/1a1c72da-99f5-4976-b608-38ee505f2b67"
 					(reference "J1")
@@
 		)
 		(instances
-			(project ""
+			(project "2Buttons_Input"
 				(path "/1a1c72da-99f5-4976-b608-38ee505f2b67"
 					(reference "SW2")
@@
 		)
 		(instances
-			(project ""
+			(project "2Buttons_Input"
 				(path "/1a1c72da-99f5-4976-b608-38ee505f2b67"
 					(reference "R1")
@@
 		)
 	)
+	(embedded_fonts no)
 )
